Commit message: Adding jackal race world and map

File: urdf/udacity_bot.xacro (robot description, xacro)
@@ -1,4 +1,5 @@
 <?xml version='1.0'?>
 <robot name="udacity_bot" xmlns:xacro="http://www.ros.org/wiki/xacro">
+  <xacro:include filename="$(find udacity_bot)/urdf/udacity_bot.gazebo" />
   <link name="robot_footprint"></link>
   <joint name="robot_footprint_joint" type="fixed">
@@ -191,5 +192,6 @@
       <origin xyz="0 0 0" rpy="0 0 0"/>
       <geometry>
-        <mesh filename="$(find udacity_bot)/meshes/hokuyo.dae"/>
+        <mesh filename="package://udacity_bot/meshes/hokuyo.dae"/>
+                <!-- mesh filename="$(find udacity_bot)/meshes/hokuyo.dae"/ -->
       </geometry>
     </visual>
