Commit message: Migrating project

File: urdf/robot_localization_ros.xacro (robot description, xacro)
@@ -1,5 +1,5 @@
 <?xml version='1.0'?>
-<robot name="udacity_bot" xmlns:xacro="http://www.ros.org/wiki/xacro">
-  <xacro:include filename="$(find udacity_bot)/urdf/udacity_bot.gazebo" />
+<robot name="robot_localization_ros" xmlns:xacro="http://www.ros.org/wiki/xacro">
+  <xacro:include filename="$(find robot_localization_ros)/urdf/robot_localization_ros.gazebo" />
   <link name="robot_footprint"></link>
   <joint name="robot_footprint_joint" type="fixed">
@@ -192,5 +192,5 @@
       <origin xyz="0 0 0" rpy="0 0 0"/>
       <geometry>
-        <mesh filename="package://udacity_bot/meshes/hokuyo.dae"/>
+        <mesh filename="package://robot_localization_ros/meshes/hokuyo.dae"/>
                 <!-- mesh filename="$(find udacity_bot)/meshes/hokuyo.dae"/ -->
       </geometry>

Commit message: feat: Robot Model and Tuning for Goal

File: urdf/robot_localization_ros.xacro (robot description, xacro)
@@ -11,5 +11,5 @@
     <pose>0 0 0.1 0 0 0</pose>
     <inertial>
-      <mass value="15.0"/>
+      <mass value="10.0"/>
       <origin xyz="0.0 0 0" rpy=" 0 0 0"/>
       <inertia
@@ -22,5 +22,5 @@
       <origin xyz="0 0 0" rpy=" 0 0 0"/>
       <geometry>
-        <box size=".4 .2 .1"/>
+        <box size=".2 .2 .1"/>
       </geometry>
     </collision>
@@ -28,7 +28,8 @@
       <origin xyz="0 0 0" rpy=" 0 0 0"/>
       <geometry>
-        <box size=".4 .2 .1"/>
-      </geometry>
-    </visual>
+        <box size=".2 .2 .1"/>
+      </geometry>
+    </visual>
+<!--
     <collision name='back_caster_collision'>
       <origin xyz="-0.15 0 -0.05" rpy=" 0 0 0"/>
@@ -53,6 +54,7 @@
       </geometry>
     </visual>
+-->
     <collision name='front_caster_collision'>
-      <origin xyz="0.15 0 -0.05" rpy=" 0 0 0"/>
+      <origin xyz="0.075 0 -0.05" rpy=" 0 0 0"/>
       <geometry>
         <sphere radius="0.05"/>
@@ -70,5 +72,5 @@
     </collision>
     <visual name='front_caster_visual'>
-      <origin xyz="0.15 0 -0.05" rpy=" 0 0 0"/>
+      <origin xyz="0.075 0 -0.05" rpy=" 0 0 0"/>
       <geometry>
         <sphere radius="0.05"/>
@@ -102,5 +104,5 @@
   <!-- left wheel joint -->
   <joint type="continuous" name="left_wheel_hinge">
-    <origin xyz="0 0.15 0" rpy="0 0 0"/>
+    <origin xyz="-0.1 0.15 0" rpy="0 0 0"/>
     <child link="left_wheel"/>
     <parent link="chassis"/>
@@ -135,5 +137,5 @@
   <!-- right wheel joint -->
   <joint type="continuous" name="right_wheel_hinge">
-    <origin xyz="0 -0.15 0" rpy="0 0 0"/>
+    <origin xyz="-0.1 -0.15 0" rpy="0 0 0"/>
     <child link="right_wheel"/>
     <parent link="chassis"/>
@@ -168,5 +170,5 @@
 <!-- Camera Joint -->
   <joint type="fixed" name="camera_joint">
-    <origin xyz="0.2 0 0" rpy="0 0 0"/>
+    <origin xyz="0.1 0 0" rpy="0 0 0"/>
     <child link="camera"/>
     <parent link="chassis"/>
@@ -199,5 +201,5 @@
 <!-- Laser Range Finder Joint -->
   <joint type="fixed" name="hokuyo_joint">
-    <origin xyz="0.15 0 0.1" rpy="0 0 0"/>
+    <origin xyz="0.0 0 0.1" rpy="0 0 0"/>
     <child link="hokuyo"/>
     <parent link="chassis"/>
